Commit message: fix home pose

File: Assets/URDF/ur10e_rg2/ur10e_rg2_description/ur10e_rg2.urdf (robot description, URDF)
Before this commit: robot ur10e_rg2, 19 links, 18 joints
Joints:
- joint robot_elbow_joint: origin xyz=-0.6127 0 0 rpy=0 0 0 -> xyz=-0.6127 0 0 rpy=0 0 20.4
- joint robot_shoulder_lift_joint: origin xyz=0 0 0 rpy=1.570796327 0 0 -> xyz=0 0 0 rpy=1.570796327 14.12 0
- joint robot_wrist_1_joint: origin xyz=-0.57155 0 0.17415 rpy=0 0 0 -> xyz=-0.57155 0 0.17415 rpy=0 0 4.7
- joint robot_wrist_2_joint: origin xyz=0 -0.11985 -2.458164590756244e-11 rpy=1.570796327 0 0 -> xyz=0 -0.11985 -2.458164590756244e-11 rpy=1.570796327 7.8 0
- joint robot_wrist_3_joint: origin xyz=0 0.11655 -2.390480459346185e-11 rpy=1.570796326589793 3.141592653589793 3.141592653589793 -> xyz=0 0.11655 -2.390480459346185e-11 rpy=1.570796326589793 80 3.141592653589793
